Commit message: init

File: src/my_simulations/models/urdf/delivery_robot.urdf (robot description, URDF)
Before this commit: robot delivery_robot, 15 links, 14 joints
Links:
- link hokuyo: geometry collision box size=0.1 0.1 0.1; visual mesh filename=package://my_simulations/models/meshes/hokuyo.dae
