Commit message: don"t know

File: src/my_simulations/models/urdf/mixed_robot.urdf (robot description, URDF)
Before this commit: robot mixed_robot, 26 links, 25 joints
Links:
- link arm_base_link: mass None -> 0.1

Commit message: controllers work!

File: src/my_simulations/models/urdf/mixed_robot.urdf (robot description, URDF)
Before this commit: robot mixed_robot, 25 links, 24 joints
Links:
- removed link base_scan
- removed link imu_link
Joints:
- removed joint base_scan_joint
- removed joint imu_joint

Commit message: controllers work but diff not!

File: src/my_simulations/models/urdf/mixed_robot.urdf (robot description, URDF)
Before this commit: robot mixed_robot, 23 links, 22 joints
Links:
- added link world
- link robot_footprint: mass None -> 3.06
Joints:
- added joint world_joint: type fixed, parent world, child robot_footprint, origin xyz=0 0 0 rpy=0 0 0

Commit message: controllers work but diff not!

File: src/my_simulations/models/urdf/mixed_robot.urdf (robot description, URDF)
Before this commit: robot mixed_robot, 24 links, 23 joints
Links:
- removed link world
- added link arm_base_link
- link robot_footprint: mass 3.06 -> None
Joints:
- removed joint world_joint
- added joint base_to_arm_joint: type fixed, parent base_chassis, child arm_base_link, origin xyz=0 0 0 rpy=0 0 0
- joint joint1: parent base_chassis -> arm_base_link
