Commit message: init

File: models/urdf/.ipynb_checkpoints/mixed_robot_2-checkpoint.urdf (robot description, URDF)
Before this commit: robot mixed_robot_2, 24 links, 23 joints
Joints:
- joint camera_joint: origin xyz=0.275 0 0.049999999999999996 rpy=0 0 0 -> xyz=0.275 0 0.1 rpy=0 0 0

Commit message: robot_2 works

File: models/urdf/.ipynb_checkpoints/mixed_robot_2-checkpoint.urdf (robot description, URDF)
Before this commit: robot mixed_robot_2, 24 links, 23 joints
Links:
- removed link base_link
- added link arm_base_link
- link link1: geometry collision cylinder length=0.10 radius=0.05; visual cylinder length=0.10 radius=0.05
Joints:
- removed joint base_link
- added joint base_link_joint: type fixed, parent base_chassis, child arm_base_link, origin xyz=0 0 0.075 rpy=0 0 0
- joint camera_joint: origin xyz=0.275 0 0.1 rpy=0 0 0 -> xyz=0.275 0 0.15 rpy=0 0 0
- joint joint1: origin xyz=0 0 0.01 rpy=0 0 0 -> xyz=0 0 0.0  rpy=0 0 0; parent base_link -> arm_base_link
- joint robot_footprint_joint: origin xyz=0 0 0 rpy=0 0 0 -> xyz=0 0 0.1175 rpy=0 0 0

File: models/urdf/mixed_robot.urdf (robot description, URDF)
Before this commit: robot mixed_robot, 25 links, 23 joints
Links:
- removed link base_link
- removed link world
- added link arm_base_link
- link hokuyo: geometry collision box size=0.1 0.1 0.1; visual mesh filename=package://my_simulations/models/meshes/hokuyo.dae
- link link1: geometry collision cylinder length=0.10 radius=0.05; visual cylinder length=0.10 radius=0.05
Joints:
- removed joint fixed
- added joint base_link_joint: type fixed, parent base_chassis, child arm_base_link, origin xyz=0 0 0.075 rpy=0 0 0
- joint camera_joint: origin xyz=0.275 0 0.049999999999999996 rpy=0 0 0 -> xyz=0.275 0 0.15 rpy=0 0 0
- joint joint1: origin xyz=0 0 0.01 rpy=0 0 0 -> xyz=0 0 0.0  rpy=0 0 0; parent base_link -> arm_base_link
- joint robot_footprint_joint: origin xyz=0 0 0 rpy=0 0 0 -> xyz=0 0 0.1175 rpy=0 0 0
