Commit message: 8_11

File: models/urdf/mixed_robot.urdf (robot description, URDF)
Before this commit: robot mixed_robot, 24 links, 23 joints
Links:
- removed link arm_base_link
- added link base_link, mass 0.1; collision cylinder length=0.02 radius=0.5
- added link world
- link hokuyo: geometry collision box size=0.1 0.1 0.1; visual mesh filename=package://my_simulation/models/meshes/hokuyo.dae
- link link1: geometry collision cylinder length=0.10 radius=0.10; visual cylinder length=0.10 radius=0.10
Joints:
- removed joint base_link_joint
- added joint fixed: type fixed, parent world, child base_link
- joint camera_joint: origin xyz=0.275 0 0.15 rpy=0 0 0 -> xyz=0.275 0 0.049999999999999996 rpy=0 0 0
- joint joint1: origin xyz=0 0 0.0  rpy=0 0 0 -> xyz=0 0 0.01 rpy=0 0 0; parent arm_base_link -> base_link
- joint robot_footprint_joint: origin xyz=0 0 0.1175 rpy=0 0 0 -> xyz=0 0 0 rpy=0 0 0

File: src/my_simulations/models/urdf/.ipynb_checkpoints/mixed_robot-checkpoint.urdf (robot description, URDF)
Before this commit: robot mixed_robot, 24 links, 23 joints
Links:
- removed link base_link
- added link arm_base_link
- added link base_scan, mass 0.001; collision box size=.001 .001 .001; visual box size=0.001 0.001 0.001
- added link imu_link, mass 0.001; collision box size=.001 .001 .001; visual box size=0.001 0.001 0.001
- link back_container_side: geometry collision box size=0.01 0.4 0.1; visual box size=0.01 0.4 0.1
- link back_left_caster: geometry collision sphere radius=0.02125; visual sphere radius=0.02125
- link back_right_caster: geometry collision sphere radius=0.02125; visual sphere radius=0.02125
- link base_chassis: geometry collision box size=0.5 0.4 0.15; visual box size=0.5 0.4 0.15
- link front_container_side: geometry collision box size=0.05 0.4 0.1; visual box size=0.05 0.4 0.1
- link front_left_caster: geometry collision sphere radius=0.02125; visual sphere radius=0.02125
- link front_right_caster: geometry collision sphere radius=0.02125; visual sphere radius=0.02125
- link left_container_side: geometry collision box size=0.5 0.01 0.1; visual box size=0.5 0.01 0.1
- link left_wheel: geometry collision cylinder length=0.02 radius=0.08; visual cylinder length=0.02 radius=0.08
- link link1: geometry collision cylinder length=0.10 radius=0.05; visual cylinder length=0.10 radius=0.05
- link link2: geometry collision cylinder length=0.30 radius=0.03; visual cylinder length=0.30 radius=0.03
- link right_container_side: geometry collision box size=0.5 0.01 0.1; visual box size=0.5 0.01 0.1
- link right_wheel: geometry collision cylinder length=0.02 radius=0.08; visual cylinder length=0.02 radius=0.08
Joints:
- removed joint fixed_arm_base
- added joint base_link_joint: type fixed, parent base_chassis, child arm_base_link, origin xyz=0 0 0.075 rpy=0 0 0
- added joint base_scan_joint: type fixed, parent base_chassis, child imu_link, origin xyz=0.25 0 0.075, axis 1 0 0
- added joint imu_joint: type fixed, parent base_chassis, child imu_link, origin xyz=0.25 0 0.1, axis 1 0 0
- joint back_container_side_hinge: origin xyz=-0.295 0.0 0.25 rpy=0 0 0 -> xyz=-0.245 0.0 0.125 rpy=0 0 0
- joint back_left_caster_hinge: origin xyz=-0.26 0.22 0.025 rpy=0 0 0 -> xyz=-0.234375 0.184375 -0.09625 rpy=0 0 0
- joint back_right_caster_hinge: origin xyz=-0.26 -0.22 0.025 rpy=0 0 0 -> xyz=-0.234375 -0.184375 -0.09625 rpy=0 0 0
- joint camera_joint: origin xyz=0.33 0 -0.04 rpy=0 0 0 -> xyz=0.275 0 0.15 rpy=0 0 0
- joint front_container_side_hinge: origin xyz=0.25 0.0 0.25 rpy=0 0 0 -> xyz=0.225 0.0 0.125 rpy=0 0 0
- joint front_left_caster_hinge: origin xyz=0.26 0.22 0.025 rpy=0 0 0 -> xyz=0.234375 0.184375 -0.09625 rpy=0 0 0
- joint front_right_caster_hinge: origin xyz=0.26 -0.22 0.025 rpy=0 0 0 -> xyz=0.234375 -0.184375 -0.09625 rpy=0 0 0
- joint hokuyo_joint: origin xyz=0.25 0 0.35 rpy=0 0 0 -> xyz=0.225 0 0.2925 rpy=0 0 0
- joint joint1: origin xyz=0 0 0.02 rpy=0 0 0 -> xyz=0 0 0.0  rpy=0 0 0; parent base_link -> arm_base_link
- joint joint2: origin xyz=0 0 0.0 rpy=0 0 0 -> xyz=0 0 0.08 rpy=0 0 0
- joint joint3: origin xyz=0 0 0.25 rpy=0 0 0 -> xyz=0 0 0.28 rpy=0 0 0
- joint joint4: origin xyz=0 0 0.6 rpy=0 0 0 -> xyz=0 0 0.28 rpy=0 0 0
- joint left_container_side_hinge: origin xyz=0.0 0.25 0.25 rpy=0 0 0 -> xyz=0.0 0.195 0.125 rpy=0 0 0
- joint left_wheel_hinge: origin xyz=0 0.26 0.09 rpy=0 0 0 -> xyz=0 0.21500000000000002 -0.0375 rpy=0 0 0
- joint right_container_side_hinge: origin xyz=0.0 -0.25 0.25 rpy=0 0 0 -> xyz=0.0 -0.195 0.125 rpy=0 0 0
- joint right_wheel_hinge: origin xyz=0 -0.26 0.09 rpy=0 0 0 -> xyz=0 -0.21500000000000002 -0.0375 rpy=0 0 0
- joint robot_footprint_joint: origin xyz=0 0 0 rpy=0 0 0 -> xyz=0 0 0.1175 rpy=0 0 0

File: src/my_simulations/models/urdf/delivery_robot.xacro (robot description, xacro)
@@ -13,5 +13,5 @@
   <xacro:property name="caster_mass" value="0.1"/>
   <!-- Include gazebo properties -->
-  <xacro:include filename="$(find my_simulations)/models/urdf/delivery_robot.gazebo" />
+  <xacro:include filename="$(find my_simulation)/models/urdf/delivery_robot.gazebo" />
   <!-- Define inertia macros  -->
   <xacro:macro name="cuboid_inertia" params="m x y z">
@@ -199,5 +199,5 @@
       <origin xyz="0 0 0" rpy=" 0 0 0"/>
       <geometry>
-        <mesh filename="package://my_simulations/models/meshes/hokuyo.dae"/>
+        <mesh filename="package://my_simulation/models/meshes/hokuyo.dae"/>
       </geometry>
     </visual>

File: src/my_simulations/models/urdf/mixed_robot.urdf (robot description, URDF)
Before this commit: robot mixed_robot, 24 links, 23 joints
Links:
- removed link base_link
- added link arm_base_link
- added link base_scan, mass 0.001; collision box size=.001 .001 .001; visual box size=0.001 0.001 0.001
- added link imu_link, mass 0.001; collision box size=.001 .001 .001; visual box size=0.001 0.001 0.001
- link back_container_side: geometry collision box size=0.01 0.4 0.1; visual box size=0.01 0.4 0.1
- link back_left_caster: geometry collision sphere radius=0.02125; visual sphere radius=0.02125
- link back_right_caster: geometry collision sphere radius=0.02125; visual sphere radius=0.02125
- link base_chassis: geometry collision box size=0.5 0.4 0.15; visual box size=0.5 0.4 0.15
- link front_container_side: geometry collision box size=0.05 0.4 0.1; visual box size=0.05 0.4 0.1
- link front_left_caster: geometry collision sphere radius=0.02125; visual sphere radius=0.02125
- link front_right_caster: geometry collision sphere radius=0.02125; visual sphere radius=0.02125
- link left_container_side: geometry collision box size=0.5 0.01 0.1; visual box size=0.5 0.01 0.1
- link left_wheel: geometry collision cylinder length=0.02 radius=0.08; visual cylinder length=0.02 radius=0.08
- link link1: geometry collision cylinder length=0.10 radius=0.05; visual cylinder length=0.10 radius=0.05
- link link2: geometry collision cylinder length=0.30 radius=0.03; visual cylinder length=0.30 radius=0.03
- link right_container_side: geometry collision box size=0.5 0.01 0.1; visual box size=0.5 0.01 0.1
- link right_wheel: geometry collision cylinder length=0.02 radius=0.08; visual cylinder length=0.02 radius=0.08
Joints:
- removed joint fixed_arm_base
- added joint base_link_joint: type fixed, parent base_chassis, child arm_base_link, origin xyz=0 0 0.075 rpy=0 0 0
- added joint base_scan_joint: type fixed, parent base_chassis, child base_scan, origin xyz=0.25 0 0.075, axis 1 0 0
- added joint imu_joint: type fixed, parent base_chassis, child imu_link, origin xyz=0.25 0 0.1, axis 1 0 0
- joint back_container_side_hinge: origin xyz=-0.295 0.0 0.25 rpy=0 0 0 -> xyz=-0.245 0.0 0.125 rpy=0 0 0
- joint back_left_caster_hinge: origin xyz=-0.26 0.22 0.025 rpy=0 0 0 -> xyz=-0.234375 0.184375 -0.09625 rpy=0 0 0
- joint back_right_caster_hinge: origin xyz=-0.26 -0.22 0.025 rpy=0 0 0 -> xyz=-0.234375 -0.184375 -0.09625 rpy=0 0 0
- joint camera_joint: origin xyz=0.33 0 -0.04 rpy=0 0 0 -> xyz=0.275 0 0.15 rpy=0 0 0
- joint front_container_side_hinge: origin xyz=0.25 0.0 0.25 rpy=0 0 0 -> xyz=0.225 0.0 0.125 rpy=0 0 0
- joint front_left_caster_hinge: origin xyz=0.26 0.22 0.025 rpy=0 0 0 -> xyz=0.234375 0.184375 -0.09625 rpy=0 0 0
- joint front_right_caster_hinge: origin xyz=0.26 -0.22 0.025 rpy=0 0 0 -> xyz=0.234375 -0.184375 -0.09625 rpy=0 0 0
- joint hokuyo_joint: origin xyz=0.25 0 0.35 rpy=0 0 0 -> xyz=0.225 0 0.225 rpy=0 0 0
- joint joint1: origin xyz=0 0 0.02 rpy=0 0 0 -> xyz=0 0 0.0  rpy=0 0 0; parent base_link -> arm_base_link
- joint joint2: origin xyz=0 0 0.0 rpy=0 0 0 -> xyz=0 0 0.08 rpy=0 0 0
- joint joint3: origin xyz=0 0 0.25 rpy=0 0 0 -> xyz=0 0 0.28 rpy=0 0 0
- joint joint4: origin xyz=0 0 0.6 rpy=0 0 0 -> xyz=0 0 0.28 rpy=0 0 0
- joint left_container_side_hinge: origin xyz=0.0 0.25 0.25 rpy=0 0 0 -> xyz=0.0 0.195 0.125 rpy=0 0 0
- joint left_wheel_hinge: origin xyz=0 0.26 0.09 rpy=0 0 0 -> xyz=0 0.21500000000000002 -0.0375 rpy=0 0 0
- joint right_container_side_hinge: origin xyz=0.0 -0.25 0.25 rpy=0 0 0 -> xyz=0.0 -0.195 0.125 rpy=0 0 0
- joint right_wheel_hinge: origin xyz=0 -0.26 0.09 rpy=0 0 0 -> xyz=0 -0.21500000000000002 -0.0375 rpy=0 0 0
- joint robot_footprint_joint: origin xyz=0 0 0 rpy=0 0 0 -> xyz=0 0 0.1175 rpy=0 0 0
