Commit message: don"t know

File: src/my_simulations/models/urdf/.ipynb_checkpoints/mixed_robot-checkpoint.urdf (robot description, URDF)
Before this commit: robot mixed_robot, 26 links, 25 joints
Links:
- removed link arm_base_link
Joints:
- removed joint base_link_joint
- joint base_scan_joint: child imu_link -> base_scan
- joint hokuyo_joint: origin xyz=0.225 0 0.2925 rpy=0 0 0 -> xyz=0.225 0 0.225 rpy=0 0 0
- joint joint1: origin xyz=0 0 0.0  rpy=0 0 0 -> xyz=0 0 0.05  rpy=0 0 0; parent arm_base_link -> base_chassis

File: src/my_simulations/models/urdf/mixed_robot.urdf (robot description, URDF)
Before this commit: robot mixed_robot, 26 links, 25 joints
Links:
- removed link arm_base_link
Joints:
- removed joint base_link_joint
- joint joint1: origin xyz=0 0 0.0  rpy=0 0 0 -> xyz=0 0 0.05  rpy=0 0 0; parent arm_base_link -> base_chassis
