Commit message: fingers inertia needs correction

File: src/robot_2/models/urdf/.ipynb_checkpoints/mixed_robot-Copy2-checkpoint.urdf (robot description, URDF)
Before this commit: robot mixed_robot, 26 links, 25 joints
Links:
- removed link base_scan
- removed link imu_link
- link arm_base_link: mass 0.1 -> None
- link hokuyo: geometry collision box size=0.1 0.1 0.1; visual mesh filename=package://robot_2/models/meshes/hokuyo.dae
Joints:
- removed joint base_link_joint
- removed joint base_scan_joint
- removed joint imu_joint
- added joint base_to_arm_joint: type fixed, parent base_chassis, child arm_base_link, origin xyz=0 0 0 rpy=0 0 0
- joint joint1: origin xyz=0 0 0.0  rpy=0 0 0 -> xyz=0 0 0.05  rpy=0 0 0

File: src/robot_2/models/urdf/.ipynb_checkpoints/mixed_robot-checkpoint.urdf (robot description, URDF)
Before this commit: robot mixed_robot, 25 links, 24 joints
Links:
- removed link base_scan
- removed link imu_link
- added link arm_base_link
- link finger1: geometry collision box size=0.06 0.01 .07; visual box size=0.06 0.01 .07
- link finger2: geometry collision box size=0.06 0.01 .07; visual box size=0.06 0.01 .07
- link hokuyo: geometry collision box size=0.1 0.1 0.1; visual mesh filename=package://robot_2/models/meshes/hokuyo.dae
Joints:
- removed joint base_scan_joint
- removed joint imu_joint
- added joint base_to_arm_joint: type fixed, parent base_chassis, child arm_base_link, origin xyz=0 0 0 rpy=0 0 0
- joint f_joint1: limit lower=0.0 upper=0.020 effort=20 velocity=0.2 -> lower=-0.005 upper=0.020 effort=20 velocity=1.0; origin xyz=0 -0.025 0.1 rpy=0 0 0 -> xyz=0 -0.025 0.11 rpy=0 0 0
- joint f_joint2: limit lower=-0.020 upper=0 effort=20 velocity=0.2 -> lower=-0.020 upper=0.005 effort=20 velocity=1.0; origin xyz=0 0.025 0.1 rpy=0 0 0 -> xyz=0 0.025 0.11 rpy=0 0 0
- joint joint1: limit (none) -> lower=-6.28319 upper=6.28319 effort=100 velocity=1; parent base_chassis -> arm_base_link; type continuous -> revolute
- joint joint2: origin xyz=0 0 0.08 rpy=0 0 0 -> xyz=0 0 0.125 rpy=0 0 0

File: src/robot_2/models/urdf/mixed_robot-Copy2.urdf (robot description, URDF)
Before this commit: robot mixed_robot, 25 links, 24 joints
Links:
- removed link base_scan
- removed link imu_link
- added link arm_base_link
- link hokuyo: geometry collision box size=0.1 0.1 0.1; visual mesh filename=package://robot_2/models/meshes/hokuyo.dae
Joints:
- removed joint base_scan_joint
- removed joint imu_joint
- added joint base_to_arm_joint: type fixed, parent base_chassis, child arm_base_link, origin xyz=0 0 0 rpy=0 0 0
- joint joint1: parent base_chassis -> arm_base_link

File: src/robot_2/models/urdf/mixed_robot.urdf (robot description, URDF)
Before this commit: robot mixed_robot, 24 links, 23 joints
Links:
- link finger1: geometry collision box size=0.06 0.01 .07; visual box size=0.06 0.01 .07
- link finger2: geometry collision box size=0.06 0.01 .07; visual box size=0.06 0.01 .07
Joints:
- joint f_joint1: limit lower=0.0 upper=0.020 effort=20 velocity=0.2 -> lower=-0.005 upper=0.020 effort=20 velocity=1.0; origin xyz=0 -0.025 0.1 rpy=0 0 0 -> xyz=0 -0.025 0.11 rpy=0 0 0
- joint f_joint2: limit lower=-0.020 upper=0 effort=20 velocity=0.2 -> lower=-0.020 upper=0.005 effort=20 velocity=1.0; origin xyz=0 0.025 0.1 rpy=0 0 0 -> xyz=0 0.025 0.11 rpy=0 0 0
- joint joint1: limit (none) -> lower=-6.28319 upper=6.28319 effort=100 velocity=1; type continuous -> revolute
- joint joint2: origin xyz=0 0 0.08 rpy=0 0 0 -> xyz=0 0 0.125 rpy=0 0 0
